File: Amiga PSU 312503-02.kicad_sch (KiCad schematic)
At the start: 38 parts, among them IC1 L296P, IC2 L4960, IC3 L7912CV (12v 1.5A), Q1 C137, SW1 SW_SPST

Commit message: Add files via upload
Update C10 to 330uF
Update Q1 to TYN058
Parts:
- C10: value 2200uF 40V -> 330uF 40V
- Q1: value C137 -> TYN058 C137
Changed lines of the file:
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@@
 			)
 		)
-		(property "Value" "C137"
+		(property "Value" "TYN058 C137"
 			(at 261.62 105.4099 0)
 			(effects
@@
 			)
 		)
-		(property "Value" "2200uF 40V"
+		(property "Value" "330uF 40V"
 			(at 119.38 165.1 0)
 			(effects

Commit message: Add files via upload
Add ouput wire colour key
Other:
- note added: "Output Wire Colours: Brown : +12V Red : 5V Black : 0V Grey : -12V Yellow : Earth/Shield"
Changed lines of the file:
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@@
+		)
+	)
+	(text "Output Wire Colours:\nBrown : +12V\nRed : 5V\nBlack : 0V\nGrey : -12V\nYellow : Earth/Shield"
+		(exclude_from_sim no)
+		(at 239.776 29.718 0)
+		(effects
+			(font
+				(size 1.27 1.27)
+			)
+			(justify left)
 		)
 	)
